File: Autonomous_PCB/Autonomous_PCB.kicad_pcb (KiCad board)
At the start: 2 copper layers, 68.6 x 53.3 mm, 24 parts, among them J1 HC-05, M1 Motor, M2 Motor, M3 Motor, M4 Motor, P1 Power, P2 Analog, P3 Digital, P4 Digital, P5 CONN_01X01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

Commit message: Add files via upload
Parts:
- C1: value CP1 -> 100uF
- R1: value ? -> 1K
- R2: value ? -> 2K
Changed lines of the file:
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@@
     (visible_elements 7FFFFFFF)
     (pcbplotparams
-      (layerselection 0x010f0_ffffffff)
+      (layerselection 0x01000_ffffffff)
       (usegerberextensions false)
       (usegerberattributes false)
@@
       (drillshape 0)
       (scaleselection 1)
-      (outputdirectory ""))
+      (outputdirectory "makerspace/"))
   )
   (net 0 "")
@@
       (effects (font (size 1 1) (thickness 0.15)))
     )
-    (fp_text value ? (at 3.81 2.37) (layer F.Fab)
+    (fp_text value 1K (at 3.81 2.37) (layer F.Fab)
       (effects (font (size 1 1) (thickness 0.15)))
     )
@@
       (effects (font (size 1 1) (thickness 0.15)))
     )
-    (fp_text value CP1 (at 2.5 6.25 90) (layer F.Fab)
+    (fp_text value 100uF (at 2.5 6.25 90) (layer F.Fab)
       (effects (font (size 1 1) (thickness 0.15)))
     )
@@
       (effects (font (size 1 1) (thickness 0.15)))
     )
-    (fp_text value ? (at 3.81 2.37) (layer F.Fab)
-      (effects (font (size 1 1) (thickness 0.15)))
-    )
+    (fp_text value 2K (at 3.81 2.37) (layer F.Fab)
+      (effects (font (size 1 1) (thickness 0.15)))
+    )

Commit message: Add files via upload
Parts:
- J1: footprint Connector_PinSocket_1.00mm:PinSocket_1x06_P1.00mm_Vertical -> 90147-1106:SHDR6W70P0X254_1X6_1524X244X870P
- moved J1 4.26 mm to (172.7, 81.3), turned to 180 degrees
Routing:
- net Net-(J1-Pad5): track 23.1 -> 26.9 mm
- net +5V: track 78.1 -> 81.1 mm
- net GND: track 254.3 -> 256.5 mm
- net /3(**): track 8.02 -> 6.45 mm
