File: Autonomous_PCB/Autonomous_PCB.sch (KiCad schematic (older format))
At the start: 13 parts, among them J1 HC-05, P1 Power, P2 Analog, P3 Digital, P4 Digital, P5 CONN_01X01, P6 CONN_01X01, P7 CONN_01X01, P8 CONN_01X01

Commit message: Add files via upload
Parts:
- added Q?: IRF3708PBF, TO254P469X1042X1967-3P, symbol IRF3708PBF:IRF3708PBF
- added R3: 100K, symbol Device:R
- R1, R2: value R -> ?
- TH1: renamed from TH?; value Thermistor -> 100K
Connections:
- net +5V: now also TH1.2
- net 8: now also Q?.1
- net A0: now also TH1.1, R3.1
- net GND: now also R3.2
Other:
- moved on the sheet: TH1
Changed lines of the file:
@@
 Wire Wire Line
 	7700 3050 8050 3050
-Wire Wire Line
-	7700 3150 8050 3150
 $Comp
 L Connector_Generic:Conn_01x10 P3
@@
 	6900 3650 6400 3650
 Wire Wire Line
-	6900 3550 6400 3550
-Wire Wire Line
 	6650 2950 6650 2500
 Wire Wire Line
@@
 L power:GND #PWR03
 U 1 1 56D70CC2
-P 6800 4200
-F 0 "#PWR03" H 6800 3950 50  0001 C CNN
-F 1 "GND" H 6800 4050 50  0000 C CNN
-F 2 "" H 6800 4200 50  0000 C CNN
-F 3 "" H 6800 4200 50  0000 C CNN
-	1    6800 4200
+P 5650 4200
+F 0 "#PWR03" H 5650 3950 50  0001 C CNN
+F 1 "GND" H 5650 4050 50  0000 C CNN
+F 2 "" H 5650 4200 50  0000 C CNN
+F 3 "" H 5650 4200 50  0000 C CNN
+	1    5650 4200
 	1    0    0    -1
 $EndComp
@@
 	7700 3550 9100 3550
 $Comp
-L Device:Thermistor TH?
+L Device:Thermistor TH1
 U 1 1 5DAB329E
-P 5450 2300
-F 0 "TH?" V 5208 2300 50  0000 C CNN
-F 1 "Thermistor" V 5299 2300 50  0000 C CNN
-F 2 "" H 5450 2300 50  0001 C CNN
-F 3 "~" H 5450 2300 50  0001 C CNN
-	1    5450 2300
+P 5500 3550
+F 0 "TH1" V 5258 3550 50  0000 C CNN
+F 1 "100K" V 5349 3550 50  0000 C CNN
+F 2 "" H 5500 3550 50  0001 C CNN
+F 3 "~" H 5500 3550 50  0001 C CNN
+	1    5500 3550
 	0    1    1    0
 $EndComp
@@
 P 8650 4200
 F 0 "R1" V 8443 4200 50  0000 C CNN
-F 1 "R" V 8534 4200 50  0000 C CNN
+F 1 "?" V 8534 4200 50  0000 C CNN
 F 2 "" V 8580 4200 50  0001 C CNN
 F 3 "~" H 8650 4200 50  0001 C CNN
@@
 P 9100 4400
 F 0 "R2" H 9170 4446 50  0000 L CNN
-F 1 "R" H 9170 4355 50  0000 L CNN
+F 1 "?" H 9170 4355 50  0000 L CNN
 F 2 "" V 9030 4400 50  0001 C CNN
 F 3 "~" H 9100 4400 50  0001 C CNN
@@
 	10050 3650 9500 3650
 Connection ~ 6550 3050
+Wire Wire Line
+	5700 3550 6100 3550
+Wire Wire Line
+	5300 3550 5300 4800
+Wire Wire Line
+	5300 4800 6550 4800
+Connection ~ 6550 4800
+Wire Wire Line
+	5650 4200 6100 4200
+$Comp
+L Device:R R3
+U 1 1 5DAD105D
+P 6100 3850
+F 0 "R3" H 6170 3896 50  0000 L CNN
+F 1 "100K" H 6170 3805 50  0000 L CNN
+F 2 "" V 6030 3850 50  0001 C CNN
+F 3 "~" H 6100 3850 50  0001 C CNN
+	1    6100 3850
+	1    0    0    -1
+$EndComp
+Wire Wire Line
+	6100 3700 6100 3550
+Connection ~ 6100 3550
+Wire Wire Line
+	6100 3550 6900 3550
+Wire Wire Line
+	6100 4000 6100 4200
+Connection ~ 6100 4200
+Wire Wire Line
+	6100 4200 6800 4200
+$Comp
+L IRF3708PBF:IRF3708PBF Q?
+U 1 1 5DAD4E46
+P 9000 1100
+F 0 "Q?" H 9430 1246 50  0000 L CNN
+F 1 "IRF3708PBF" H 9430 1155 50  0000 L CNN
+F 2 "TO254P469X1042X1967-3P" H 9450 1050 50  0001 L CNN
+F 3 "https://componentsearchengine.com/Datasheets/1/IRF3708PBF.pdf" H 9450 950 50  0001 L CNN
+F 4 "IRF3708PBF N-Channel MOSFET, 62 A, 30 V HEXFET, 3-Pin TO-220AB Infineon" H 9450 850 50  0001 L CNN "Description"
+F 5 "4.69" H 9450 750 50  0001 L CNN "Height"
+F 6 "942-IRF3708PBF" H 9450 650 50  0001 L CNN "Mouser Part Number"
+F 7 "https://www.mouser.com/Search/Refine.aspx?Keyword=942-IRF3708PBF" H 9450 550 50  0001 L CNN "Mouser Price/Stock"
+F 8 "Infineon" H 9450 450 50  0001 L CNN "Manufacturer_Name"
+F 9 "IRF3708PBF" H 9450 350 50  0001 L CNN "Manufacturer_Part_Number"
+	1    9000 1100
+	1    0    0    -1
+$EndComp
+Wire Wire Line
+	9000 1100 8800 1100
+Wire Wire Line
+	8800 1100 8800 3150
+Wire Wire Line
+	7700 3150 8800 3150
 $EndSCHEMATC

Commit message: Add files via upload
Parts:
- added C1: CP1, Capacitor_THT:CP_Radial_D10.0mm_P5.00mm, symbol Device:CP1
- added H1: Hot End -ve, MountingHole:MountingHole_2.2mm_M2_DIN965_Pad, symbol Mechanical:MountingHole_Pad
- added H2: Hot End +ve, MountingHole:MountingHole_2.2mm_M2_DIN965_Pad, symbol Mechanical:MountingHole_Pad
- added M1, M2, M3, M4: Motor, MountingHole:MountingHole_2.2mm_M2_DIN965_Pad, symbol Mechanical:MountingHole_Pad
- added PW1: PSU +ve, MountingHole:MountingHole_2.2mm_M2_DIN965_Pad, symbol Mechanical:MountingHole_Pad
- added PW2: PSU -ve, MountingHole:MountingHole_2.2mm_M2_DIN965_Pad, symbol Mechanical:MountingHole_Pad
- J1: footprint (none) -> Connector_PinHeader_1.00mm:PinHeader_1x06_P1.00mm_Horizontal
- Q1: renamed from Q?; footprint TO254P469X1042X1967-3P -> IRF3708PBF:TO254P469X1042X1967-3P
- R1, R2, R3: footprint (none) -> Resistor_THT:R_Axial_DIN0207_L6.3mm_D2.5mm_P7.62mm_Horizontal
- TH1: footprint (none) -> Resistor_THT:R_Axial_DIN0204_L3.6mm_D1.6mm_P5.08mm_Horizontal
- gave numbers to parts that had none: 1
Connections:
- net GND: now also A1.1 (GND), A1.7 (GND), Q1.3, C1.2, PW2.1
- net at A1.3 (1B): now also M1.1
- net at A1.4 (1A): now also M2.1
- net at A1.5 (2A): now also M3.1
- net at A1.6 (2B): now also M4.1
- net at A1.8 (VMOT): now also C1.1, H2.1, PW1.1
- net at Q1.2: now also H1.1
Changed lines of the file:
@@
 $EndDescr
 $Comp
-L Driver_Motor:Pololu_Breakout_A4988 A?
+L Driver_Motor:Pololu_Breakout_A4988 A1
 U 1 1 5DA655EE
 P 9600 2300
-F 0 "A?" H 9650 1319 50  0000 C CNN
+F 0 "A1" H 9650 1319 50  0000 C CNN
 F 1 "Pololu_Breakout_A4988" H 9650 1410 50  0000 C CNN
 F 2 "Module:Pololu_Breakout-16_15.2x20.3mm" H 9875 1550 50  0001 L CNN
@@
 F 0 "TH1" V 5258 3550 50  0000 C CNN
 F 1 "100K" V 5349 3550 50  0000 C CNN
-F 2 "" H 5500 3550 50  0001 C CNN
+F 2 "Resistor_THT:R_Axial_DIN0204_L3.6mm_D1.6mm_P5.08mm_Horizontal" H 5500 3550 50  0001 C CNN
 F 3 "~" H 5500 3550 50  0001 C CNN
 	1    5500 3550
@@
 F 0 "J1" H 9850 4100 50  0000 L CNN
 F 1 "HC-05" H 9550 4100 50  0000 L CNN
-F 2 "" H 9700 3750 50  0001 C CNN
+F 2 "Connector_PinHeader_1.00mm:PinHeader_1x06_P1.00mm_Horizontal" H 9700 3750 50  0001 C CNN
 F 3 "~" H 9700 3750 50  0001 C CNN
 	1    9700 3750
@@
 F 0 "R1" V 8443 4200 50  0000 C CNN
 F 1 "?" V 8534 4200 50  0000 C CNN
-F 2 "" V 8580 4200 50  0001 C CNN
+F 2 "Resistor_THT:R_Axial_DIN0207_L6.3mm_D2.5mm_P7.62mm_Horizontal" V 8580 4200 50  0001 C CNN
 F 3 "~" H 8650 4200 50  0001 C CNN
 	1    8650 4200
@@
 Connection ~ 7800 4200
 $Comp
-L power:GND #PWR?
+L power:GND #PWR0101
 U 1 1 5DAC1976
 P 9400 4600
-F 0 "#PWR?" H 9400 4350 50  0001 C CNN
+F 0 "#PWR0101" H 9400 4350 50  0001 C CNN
 F 1 "GND" H 9405 4427 50  0000 C CNN
 F 2 "" H 9400 4600 50  0001 C CNN
@@
 F 0 "R2" H 9170 4446 50  0000 L CNN
 F 1 "?" H 9170 4355 50  0000 L CNN
-F 2 "" V 9030 4400 50  0001 C CNN
+F 2 "Resistor_THT:R_Axial_DIN0207_L6.3mm_D2.5mm_P7.62mm_Horizontal" V 9030 4400 50  0001 C CNN
 F 3 "~" H 9100 4400 50  0001 C CNN
 	1    9100 4400
@@
 	9100 4600 9400 4600
 Wire Wire Line
-	9500 3750 8850 3750
+	9500 3750 9350 3750
 Wire Wire Line
 	8850 3750 8850 4600
@@
 F 0 "R3" H 6170 3896 50  0000 L CNN
 F 1 "100K" H 6170 3805 50  0000 L CNN
-F 2 "" V 6030 3850 50  0001 C CNN
+F 2 "Resistor_THT:R_Axial_DIN0207_L6.3mm_D2.5mm_P7.62mm_Horizontal" V 6030 3850 50  0001 C CNN
 F 3 "~" H 6100 3850 50  0001 C CNN
 	1    6100 3850
@@
 	6100 4200 6800 4200
 $Comp
-L IRF3708PBF:IRF3708PBF Q?
+L IRF3708PBF:IRF3708PBF Q1
 U 1 1 5DAD4E46
 P 9000 1100
-F 0 "Q?" H 9430 1246 50  0000 L CNN
+F 0 "Q1" H 9430 1246 50  0000 L CNN
 F 1 "IRF3708PBF" H 9430 1155 50  0000 L CNN
-F 2 "TO254P469X1042X1967-3P" H 9450 1050 50  0001 L CNN
+F 2 "IRF3708PBF:TO254P469X1042X1967-3P" H 9450 1050 50  0001 L CNN
 F 3 "https://componentsearchengine.com/Datasheets/1/IRF3708PBF.pdf" H 9450 950 50  0001 L CNN
 F 4 "IRF3708PBF N-Channel MOSFET, 62 A, 30 V HEXFET, 3-Pin TO-220AB Infineon" H 9450 850 50  0001 L CNN "Description"
@@
 Wire Wire Line
 	7700 3150 8800 3150
+Wire Wire Line
+	7800 2550 7800 1300
+Wire Wire Line
+	7800 1300 9300 1300
+Connection ~ 7800 2550
+$Comp
+L Mechanical:MountingHole_Pad M1
+U 1 1 5DAA30D8
+P 10700 1850
+F 0 "M1" V 10654 2000 50  0000 L CNN
+F 1 "Motor" V 10745 2000 50  0000 L CNN
+F 2 "MountingHole:MountingHole_2.2mm_M2_DIN965_Pad" H 10700 1850 50  0001 C CNN
+F 3 "~" H 10700 1850 50  0001 C CNN
+	1    10700 1850
+	0    1    1    0
+$EndComp
+Wire Wire Line
+	10100 2300 10500 2300
+Wire Wire Line
+	10500 2300 10500 2100
+Wire Wire Line
+	10500 2100 10600 2100
+Wire Wire Line
+	10100 2200 10350 2200
+Wire Wire Line
+	10350 2200 10350 1850
+Wire Wire Line
+	10350 1850 10600 1850
+Wire Wire Line
+	10100 2400 10500 2400
+Wire Wire Line
+	10500 2400 10500 2600
+Wire Wire Line
+	10500 2600 10600 2600
+Wire Wire Line
+	10100 2500 10350 2500
+Wire Wire Line
+	10350 2500 10350 2850
+Wire Wire Line
+	10350 2850 10600 2850
+$Comp
+L Mechanical:MountingHole_Pad M2
+U 1 1 5DAAD8B3
+P 10700 2100
+F 0 "M2" V 10654 2250 50  0000 L CNN
+F 1 "Motor" V 10745 2250 50  0000 L CNN
+F 2 "MountingHole:MountingHole_2.2mm_M2_DIN965_Pad" H 10700 2100 50  0001 C CNN
+F 3 "~" H 10700 2100 50  0001 C CNN
+	1    10700 2100
+	0    1    1    0
+$EndComp
+$Comp
+L Mechanical:MountingHole_Pad M3
+U 1 1 5DAADB93
+P 10700 2600
+F 0 "M3" V 10654 2750 50  0000 L CNN
+F 1 "Motor" V 10745 2750 50  0000 L CNN
+F 2 "MountingHole:MountingHole_2.2mm_M2_DIN965_Pad" H 10700 2600 50  0001 C CNN
+F 3 "~" H 10700 2600 50  0001 C CNN
+	1    10700 2600
+	0    1    1    0
+$EndComp
+$Comp
+L Mechanical:MountingHole_Pad M4
+U 1 1 5DAADF60
+P 10700 2850
+F 0 "M4" V 10654 3000 50  0000 L CNN
+F 1 "Motor" V 10745 3000 50  0000 L CNN
+F 2 "MountingHole:MountingHole_2.2mm_M2_DIN965_Pad" H 10700 2850 50  0001 C CNN
+F 3 "~" H 10700 2850 50  0001 C CNN
+	1    10700 2850
+	0    1    1    0
+$EndComp
+Wire Wire Line
+	9600 3100 9200 3100
+Wire Wire Line
+	9200 3100 9200 3750
+Connection ~ 9200 3750
+Wire Wire Line
+	9200 3750 8850 3750
+Wire Wire Line
+	9800 3100 9800 3250
+Wire Wire Line
+	9800 3250 9350 3250
+Wire Wire Line
+	9350 3250 9350 3750
+Connection ~ 9350 3750
+Wire Wire Line
+	9350 3750 9200 3750
+$Comp
+L Mechanical:MountingHole_Pad H1
+U 1 1 5DAB5A90
+P 8400 800
+F 0 "H1" V 8637 803 50  0000 C CNN
+F 1 "Hot End -ve" V 8546 803 50  0000 C CNN
+F 2 "MountingHole:MountingHole_2.2mm_M2_DIN965_Pad" H 8400 800 50  0001 C CNN
+F 3 "~" H 8400 800 50  0001 C CNN
+	1    8400 800
+	0    -1   -1   0
+$EndComp
+Wire Wire Line
+	8500 800  9200 800
+Wire Wire Line
+	9200 800  9200 700
+Wire Wire Line
+	9200 700  9300 700
+$Comp
+L Mechanical:MountingHole_Pad H2
+U 1 1 5DAB97DD
+P 10600 600
+F 0 "H2" V 10554 750 50  0000 L CNN
+F 1 "Hot End +ve" V 10645 750 50  0000 L CNN
+F 2 "MountingHole:MountingHole_2.2mm_M2_DIN965_Pad" H 10600 600 50  0001 C CNN
+F 3 "~" H 10600 600 50  0001 C CNN
+	1    10600 600
+	0    1    1    0
+$EndComp
+Wire Wire Line
+	9300 1300 10000 1300
+Wire Wire Line
+	10950 1300 10950 1450
+Connection ~ 9300 1300
+$Comp
+L power:GND #PWR0102
+U 1 1 5DAC0B3D
+P 10950 1450
+F 0 "#PWR0102" H 10950 1200 50  0001 C CNN
+F 1 "GND" H 10955 1277 50  0000 C CNN
+F 2 "" H 10950 1450 50  0001 C CNN
+F 3 "" H 10950 1450 50  0001 C CNN
+	1    10950 1450
+	1    0    0    -1
+$EndComp
+$Comp
+L Device:CP1 C1
+U 1 1 5DAC7741
+P 10000 1150
+F 0 "C1" H 10115 1196 50  0000 L CNN
+F 1 "CP1" H 10115 1105 50  0000 L CNN
+F 2 "Capacitor_THT:CP_Radial_D10.0mm_P5.00mm" H 10000 1150 50  0001 C CNN
+F 3 "~" H 10000 1150 50  0001 C CNN
+	1    10000 1150
+	1    0    0    -1
+$EndComp
+Wire Wire Line
+	9800 1600 9800 600
+Wire Wire Line
+	9800 600  10000 600
+Connection ~ 10000 1300
+Wire Wire Line
+	10000 1300 10400 1300
+Wire Wire Line
+	10000 600  10000 1000
+Connection ~ 10000 600
+Wire Wire Line
+	10000 600  10300 600
+$Comp
+L Mechanical:MountingHole_Pad PW1
+U 1 1 5DAD498A
+P 10300 700
+F 0 "PW1" H 10200 657 50  0000 R CNN
+F 1 "PSU +ve" H 10200 748 50  0000 R CNN
+F 2 "MountingHole:MountingHole_2.2mm_M2_DIN965_Pad" H 10300 700 50  0001 C CNN
+F 3 "~" H 10300 700 50  0001 C CNN
+	1    10300 700
+	-1   0    0    1
+$EndComp
+Connection ~ 10300 600
+Wire Wire Line
+	10300 600  10500 600
+$Comp
+L Mechanical:MountingHole_Pad PW2
+U 1 1 5DAD559A
+P 10400 1200
+F 0 "PW2" H 10500 1249 50  0000 L CNN
+F 1 "PSU -ve" H 10500 1158 50  0000 L CNN
+F 2 "MountingHole:MountingHole_2.2mm_M2_DIN965_Pad" H 10400 1200 50  0001 C CNN
+F 3 "~" H 10400 1200 50  0001 C CNN
+	1    10400 1200
+	1    0    0    -1
+$EndComp
+Connection ~ 10400 1300
+Wire Wire Line
+	10400 1300 10950 1300
 $EndSCHEMATC

Commit message: Add files via upload
Parts:
- C1: value CP1 -> 100uF
- R1: value ? -> 1K
- R2: value ? -> 2K
Changed lines of the file:
@@
 P 8650 4200
 F 0 "R1" V 8443 4200 50  0000 C CNN
-F 1 "?" V 8534 4200 50  0000 C CNN
+F 1 "1K" V 8534 4200 50  0000 C CNN
 F 2 "Resistor_THT:R_Axial_DIN0207_L6.3mm_D2.5mm_P7.62mm_Horizontal" V 8580 4200 50  0001 C CNN
 F 3 "~" H 8650 4200 50  0001 C CNN
@@
 P 9100 4400
 F 0 "R2" H 9170 4446 50  0000 L CNN
-F 1 "?" H 9170 4355 50  0000 L CNN
+F 1 "2K" H 9170 4355 50  0000 L CNN
 F 2 "Resistor_THT:R_Axial_DIN0207_L6.3mm_D2.5mm_P7.62mm_Horizontal" V 9030 4400 50  0001 C CNN
 F 3 "~" H 9100 4400 50  0001 C CNN
@@
 P 10000 1150
 F 0 "C1" H 10115 1196 50  0000 L CNN
-F 1 "CP1" H 10115 1105 50  0000 L CNN
+F 1 "100uF" H 10115 1105 50  0000 L CNN
 F 2 "Capacitor_THT:CP_Radial_D10.0mm_P5.00mm" H 10000 1150 50  0001 C CNN
 F 3 "~" H 10000 1150 50  0001 C CNN

Commit message: Add files via upload
Parts:
- J1: footprint Connector_PinHeader_1.00mm:PinHeader_1x06_P1.00mm_Horizontal -> 90147-1106:SHDR6W70P0X254_1X6_1524X244X870P
Changed lines of the file:
@@
 F 0 "J1" H 9850 4100 50  0000 L CNN
 F 1 "HC-05" H 9550 4100 50  0000 L CNN
-F 2 "Connector_PinHeader_1.00mm:PinHeader_1x06_P1.00mm_Horizontal" H 9700 3750 50  0001 C CNN
+F 2 "90147-1106:SHDR6W70P0X254_1X6_1524X244X870P" H 9700 3750 50  0001 C CNN
 F 3 "~" H 9700 3750 50  0001 C CNN
 	1    9700 3750
